File: AFR Meter/PCB Files/Screen/172x320 Screen.brd (EAGLE design)
At the start: 43.6 x 19.5 mm, 20 parts, among them IC1 CD74HC4050PWRG4, X2 FH12-12S-0.5SH

Commit message: Add files via upload
Parts:
- moved X2 6.86 mm to (18.1, 8.61), turned to 90 degrees
Routing:
- net MOSI3V3: track 6.89 -> 13.7 mm
- net CLK3V3: track 7.36 -> 9.82 mm
- net GND: track 73.4 -> 71.6 mm
- net LEDK: track 19.6 -> 18.1 mm
- net CS3V3: track 8.52 -> 7.39 mm
- net +5V: track 39.3 -> 38.3 mm
- net SPI_MOSI: track 13.4 -> 14.2 mm
Other:
- board text added: "12"
