File: Boost Gauge/PCB Files/Boost Gauge MainBoard.brd (EAGLE design)
At the start: 88 x 63 mm, 76 parts, among them IC1 MCT6SD, IC2 MCP96RL00-E_MX, IC4 ATMEGA328PB-AN, IC6 7805DT, IC7 MCP25625-E_SS, Q1 BUK7Y6R0-60EX

Commit message: v0.2 PCB
Parts:
- removed IC1: MCT6SD, MCT6SD:SOP254P1016X385-8N
- added Q2, Q3: BC817-40LT1SMD, transistor-npn:SOT23-BEC
- added R15, R16: 100k, rcl:R0805
- moved R2 10.7 mm to (46.6, 20.2), turned to 0 degrees
- moved R3 10.5 mm to (40.2, 20.2), turned to 180 degrees
- moved R6 6.35 mm to (48.5, 29.0), turned to 180 degrees
- moved R4 4.67 mm to (41.6, 29.0), turned to 180 degrees
- moved C17 3.94 mm to (40.2, 17.8), turned to 0 degrees
- moved C18 3.35 mm to (46.6, 17.8)
Connections:
- removed net N$2: IC1.2, R2.2
- new net N$4: Q3.B, R16.1, R2.1
- net +5V: now also Q2.C, Q3.C; no longer R4.2, R6.2
- net GND: now also R15.2, R16.2, R4.1, R6.1; no longer IC1.5, IC1.8, R2.1, R3.1
- net N$3: now also Q2.B, R15.1, R3.1; no longer IC1.3, R3.2
- net RPM_ISO: now also Q2.E, R4.2; no longer IC1.6, R6.1
- net RPM_SIGNAL: now also R3.2; no longer IC1.1
- net TACH_ISO: now also Q3.E, R6.2; no longer IC1.7, R4.1
- net TACH_SIGNAL: now also R2.2; no longer IC1.4
Routing:
- net +5V: track 296.0 -> 309.3 mm
- net N$4: track 0.00 -> 8.52 mm
- net N$2: track 8.17 -> 0.00 mm
- net RPM_ISO: track 22.0 -> 17.0 mm
- net TACH_ISO: track 28.0 -> 32.4 mm
- net RPM_SIGNAL: track 9.54 -> 6.66 mm
- net TACH_SIGNAL: track 9.16 -> 7.10 mm
- net N$3: track 8.18 -> 7.34 mm
- net CAN_H: track 34.0 -> 34.6 mm

Commit message: V1.0 of the mainboard files
Parts:
- removed IC6: 7805DT, linear:TO252
- added IC1: MC7805CD2TR4G, MC7805CD2TR4G:MC7805CD2TR4G
- moved C3 4.47 mm to (81.4, 42.2)
- moved C2 2.02 mm to (73.6, 46.9)
- moved D2 1.97 mm to (85.8, 34.7)
- moved C4 0.64 mm to (24.7, 17.4)
- moved C5 0.64 mm to (29.7, 22.2)
- moved IC2 0.64 mm to (24.8, 21.8)
- moved R10 0.64 mm to (17.5, 22.8)
- moved R11 0.64 mm to (17.4, 20.3)
- moved R12 0.64 mm to (29.6, 17.4)
- moved R13 0.64 mm to (19.9, 17.4)
- moved R14 0.64 mm to (17.5, 25.2)
- moved TGND 0.64 mm to (33.1, 16.5)
Connections:
- net +5V: now also IC1.3; no longer IC6.2
- net GND: now also IC1.2; no longer IC6.3
- net N$6: now also IC1.1; no longer IC6.1
Routing:
- net BOOST_CTRL_PWM: track 12.8 -> 16.4 mm, vias 64 -> 0
- net +5V: track 309.3 -> 312.4 mm
- net NTC_IN: track 28.5 -> 31.0 mm
- net N$6: track 20.5 -> 22.1 mm
- net GND: track 157.8 -> 156.5 mm, vias 133 -> 159
- net CAN_H: track 34.6 -> 35.7 mm
- net CAN_L: track 37.5 -> 36.7 mm
- net BOOST_CTRL: track 5.04 -> 5.82 mm
- net SCL: track 19.2 -> 19.8 mm
- net SDA: track 20.7 -> 21.3 mm
- removed copper zone on layer 16, net BOOST_CTRL_PWM

Commit message: Small fixes v0.2
Routing:
- net +12V: track 53.1 -> 48.3 mm
- net GND: track 156.5 -> 160.5 mm
- net +5V: track 312.4 -> 309.9 mm
Other:
- board text added: "OpenTG Boost Controller Mainboard By Kostas Anes HRD v0.2"
- board text removed: "OpenTG Boost Controller Mainboard By Kostas Anes HRD v0.1"
