File: AFR Meter/PCB Files/LSU 4.9 OpenAFR MainBoard.sch (EAGLE design)
At the start: 82 parts, among them IC2 LMV321M5X, IC3 MCP4725A2T-E_CH, IC4 ATMEGA328PB-AN, IC5 ISO6520DR, IC6 7805DT, IC7 MCP25625-E_SS, Q1 BUK7Y6R0-60EX

Commit message: Mainboard power supply and QoL updates.
Parts:
- removed C2, C4: 10uF, rcl:CPOL-EUUD-5X5,8
- removed IC6: 7805DT, linear:7805DT
- added C28: 10uF, rcl:C-EUC0805
- added C29, C30: (no value), rcl:CPOL-EU153CLV-0605
- added IC1: MC7805CD2TR4G, MC7805CD2TR4G:MC7805CD2TR4G
Connections:
- new net N$4: C21.1, RESET.1
- net +5V: now also C29.+, IC1.OUTPUT; no longer C4.+, IC6.VO
- net 5V_ISO: now also C28.1
- net GND: now also C29.-, C30.-, IC1.GROUND; no longer C2.-, C4.-, IC6.GND
- net N$6: now also C30.+, IC1.INPUT; no longer C2.+, IC6.VI
- net NRBND_GND: now also C28.2
- net RESET: no longer C21.1, RESET.1, SV1.5
Other:
- moved on the sheet: C3, D2, RESET
