File: KLT120/KLT120.kicad_sch (KiCad schematic)
At the start: 34 parts, among them IC1 LM393BIPWR, IC2 LM393BIPWR, Q1 2N7002K, Q2 2N7002K

Commit message: v0.11
Parts:
- added 111: (no value), 3_pins:90-2, symbol 3_pins:TERMINAL_2PINS
- added R22, R23: 4K7, cap_mult_pins:M0805, symbol cap_mult_pins:R-EU_M0805
Connections:
- net +3V3: now also R22.2, R23.2
- net RX: no longer IC2.7 (2OUT)
- net TX: no longer IC2.2 (1IN-)
- net L_LINE_OUT: now reaches 1.2, R21.1
- net L_LINE_OUT: now also Q2.3 (D)
- net K_LINE_OUT: now reaches 1.1, R18.1, R6.1
- net K_LINE_OUT: now also IC1.5 (2IN+), Q1.3 (D)
- net K_LINE renamed K_LINE_IN
- net K_LINE_IN: no longer IC1.5 (2IN+), Q1.3 (D)
- net L_LINE renamed L_LINE_IN
- net L_LINE_IN: no longer Q2.3 (D)
- new net RX_L: 111.1, IC2.7 (2OUT), R23.1
- new net TX_L: 111.2, IC2.2 (1IN-), R22.1
Other:
- note added: "Input Connectors"
- note added: "Logic Stage"
- note added: "MCU Connectors"
- note added: "Output Drivers"
- company: (none) -> Standalone K/L Line Transceiver for 5/3.3V MCUs
- title: (none) -> KLT120
- moved on the sheet: 1, 11, C1, C2, C3, C4, D1, IC1, IC2, PS1, Q1, Q2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

Commit message: Added PCB
Parts:
- removed 1, 11 (x2), 111: (no value), 3_pins:90-2, symbol 3_pins:TERMINAL_2PINS
- added J1, J2, J3, J4: 282812-2, 282812:2828122, symbol 282812:282812-2
- C1, C3, C4: footprint (none) -> Capacitor_SMD:C_0805_2012Metric
- C2: footprint (none) -> Capacitor_SMD:CP_Elec_5x5.7
- IC1, IC2: footprint SOP65P640X120-8N -> LM393BIPWR:SOP65P640X120-8N
- PS1: footprint SOT95P237X112-3N -> LIB_TLV76050DBZR:SOT95P237X112-3N
- R1, R10, R11, R12, R13, R14, R15, R16, R17, R18, R19, R2, R20, R21, R22, R23, R3, R4, R7, R9: footprint cap_mult_pins:M0805 -> Resistor_SMD:R_0805_2012Metric_Pad1.20x1.40mm_HandSolder
- R5, R6, R8: footprint cap_mult_pins:M1206 -> Resistor_SMD:R_1206_3216Metric_Pad1.30x1.75mm_HandSolder
Connections:
- net +12V: now also J2.1
- net GND: now also J2.2
- net K_LINE_IN: now also IC1.5 (2IN+)
- net K_LINE_OUT: now also J1.1; no longer IC1.5 (2IN+)
- net L_LINE_OUT: now also J1.2
- net RX: now also J4.1
- net RX_L: now also J3.1
- net TX: now also J4.2
- net TX_L: now also J3.2
Other:
- note added: "3.3/5V Power Supply"
- moved on the sheet: D1, R10, R11, R22, R23
